Commit message: Adding inertial tags and collision tags to the URDF files for the rail, arm, and soft gripper. This is necessary for proper physics simulation in Gazebo and other simulators that require these properties for accurate dynamics and collision detection. Also did simple gazebo launch file to test the robot in Gazebo.

File: harvest_description/urdf/mech/harvest_arm.urdf.xacro (robot description, xacro)
@@ -2,81 +2,134 @@
 <robot xmlns:xacro="http://www.ros.org/wiki/xacro">
 	<xacro:macro name="harvest_arm" params="parent_link">
+		  <!-- ARM STRUCTURE -->
+		<!-- The arm is attached to the rail carriage through base_link. -->
+		<link name="base_link">
+			<visual>
+			<geometry><cylinder radius="0.1" length="0.1"/></geometry>
+			<material name="blue"/>
+			</visual>
+			<collision>
+			<geometry><cylinder radius="0.1" length="0.1"/></geometry>
+			</collision>
+			<!-- Solid motor base carriage housing (5 kg) -->
+			<xacro:cylinder_inertial mass="5.0" radius="0.1" length="0.1">
+			<origin xyz="0 0 0" rpy="0 0 0"/>
+			</xacro:cylinder_inertial>
+		</link>
+		<!-- 2. Base Revolute Joint (Yaw) -->
+		<joint name="base_joint" type="revolute">
+			<parent link="base_link"/>
+			<child link="shoulder_link"/>
+			<axis xyz="0 0 1"/>
+			<limit lower="-3.14" upper="3.14" effort="150.0" velocity="1.0"/>
+			<origin xyz="0 0 0.05" rpy="0 0 0"/>
+			<dynamics damping="5.0" friction="2.0"/>
+		</joint>
 		<link name="shoulder_link">
 			<visual>
-				<origin xyz="0 0 0.2" rpy="0 0 0"/>
-				<geometry>
-					<cylinder radius="0.05" length="0.4"/>
-				</geometry>
-				<material name="silver"/>
+			<origin xyz="0 0 0.2" rpy="0 0 0"/>
+			<geometry><cylinder radius="0.05" length="0.4"/></geometry>
+			<material name="silver"/>
 			</visual>
+			<collision>
+			<origin xyz="0 0 0.2" rpy="0 0 0"/>
+			<geometry><cylinder radius="0.05" length="0.4"/></geometry>
+			</collision>
+			<!-- Carbon fiber/aluminum lightweight link (2.5 kg) -->
+			<xacro:cylinder_inertial mass="2.5" radius="0.05" length="0.4">
+			<origin xyz="0 0 0.2" rpy="0 0 0"/>
+			</xacro:cylinder_inertial>
 		</link>
-		<joint name="base_joint" type="revolute">
-			<parent link="${parent_link}"/>
-			<child link="shoulder_link"/>
-			<axis xyz="0 0 1"/>
-			<limit lower="-3.14" upper="3.14" effort="100.0" velocity="1.0"/>
-			<origin xyz="0 0 0.05" rpy="0 0 0"/>
-		</joint>
-		<link name="elbow_link">
-			<visual>
-				<origin xyz="0 0 0.2" rpy="0 0 0"/>
-				<geometry>
-					<cylinder radius="0.04" length="0.4"/>
-				</geometry>
-				<material name="silver"/>
-			</visual>
-		</link>
+		<!-- 3. Shoulder Revolute Joint (Pitch) -->
 		<joint name="shoulder_joint" type="revolute">
 			<parent link="shoulder_link"/>
 			<child link="elbow_link"/>
 			<axis xyz="0 1 0"/>
-			<limit lower="-1.57" upper="1.57" effort="100.0" velocity="1.0"/>
+			<limit lower="-1.57" upper="1.57" effort="150.0" velocity="1.0"/>
 			<origin xyz="0 0 0.4" rpy="0 0 0"/>
+			<dynamics damping="5.0" friction="2.0"/>
 		</joint>
-		<link name="wrist_pitch_link">
+		<link name="elbow_link">
 			<visual>
-				<geometry>
-					<cylinder radius="0.03" length="0.06"/>
-				</geometry>
-				<material name="blue"/>
+			<origin xyz="0 0 0.2" rpy="0 0 0"/>
+			<geometry><cylinder radius="0.04" length="0.4"/></geometry>
+			<material name="silver"/>
 			</visual>
+			<collision>
+			<origin xyz="0 0 0.2" rpy="0 0 0"/>
+			<geometry><cylinder radius="0.04" length="0.4"/></geometry>
+			</collision>
+			<!-- Upper arm link (2.0 kg) -->
+			<xacro:cylinder_inertial mass="2.0" radius="0.04" length="0.4">
+			<origin xyz="0 0 0.2" rpy="0 0 0"/>
+			</xacro:cylinder_inertial>
 		</link>
+		<!-- 4. Elbow Revolute Joint (Pitch) -->
 		<joint name="elbow_joint" type="revolute">
 			<parent link="elbow_link"/>
-			<child link="wrist_pitch_link"/>
+			<child xacro:name="wrist_pitch_link" link="wrist_pitch_link"/>
 			<axis xyz="0 1 0"/>
 			<limit lower="-2.0" upper="2.0" effort="100.0" velocity="1.0"/>
 			<origin xyz="0 0 0.4" rpy="0 0 0"/>
+			<dynamics damping="3.0" friction="1.0"/>
 		</joint>
-		<link name="wrist_roll_link">
+		<!-- ================= Universal Wrist (Pitch-Roll) ================= -->
+		<link name="wrist_pitch_link">
 			<visual>
-				<geometry>
-					<cylinder radius="0.03" length="0.04"/>
-				</geometry>
-				<material name="green"/>
+			<geometry><cylinder radius="0.03" length="0.06"/></geometry>
+			<material name="blue"/>
 			</visual>
+			<collision>
+			<geometry><cylinder radius="0.03" length="0.06"/></geometry>
+			</collision>
+			<!-- Small pitch motor housing (0.8 kg) -->
+			<xacro:cylinder_inertial mass="0.8" radius="0.03" length="0.06">
+			<origin xyz="0 0 0" rpy="0 0 0"/>
+			</xacro:cylinder_inertial>
 		</link>
+		<!-- 5. Wrist Joint 1 (Pitch) -->
 		<joint name="wrist_pitch_joint" type="revolute">
 			<parent link="wrist_pitch_link"/>
 			<child link="wrist_roll_link"/>
 			<axis xyz="0 1 0"/>
-			<limit lower="-1.57" upper="1.57" effort="50.0" velocity="1.5"/>
+			<limit lower="-1.57" upper="1.57" effort="40.0" velocity="1.5"/>
 			<origin xyz="0 0 0.05" rpy="0 0 0"/>
+			<dynamics damping="1.0" friction="0.5"/>
 		</joint>
-		<link name="end_effector_tool_mount">
+		<link name="wrist_roll_link">
 			<visual>
-				<geometry>
-					<cylinder radius="0.05" length="0.02"/>
-				</geometry>
-				<material name="blue"/>
+			<geometry><cylinder radius="0.03" length="0.04"/></geometry>
+			<material name="green"/>
 			</visual>
+			<collision>
+			<geometry><cylinder radius="0.03" length="0.04"/></geometry>
+			</collision>
+			<!-- Small roll motor housing (0.5 kg) -->
+			<xacro:cylinder_inertial mass="0.5" radius="0.03" length="0.04">
+			<origin xyz="0 0 0" rpy="0 0 0"/>
+			</xacro:cylinder_inertial>
 		</link>
+		<!-- 6. Wrist Joint 2 (Roll) -->
 		<joint name="wrist_roll_joint" type="revolute">
 			<parent link="wrist_roll_link"/>
 			<child link="end_effector_tool_mount"/>
 			<axis xyz="0 0 1"/>
-			<limit lower="-3.14" upper="3.14" effort="50.0" velocity="1.5"/>
+			<limit lower="-3.14" upper="3.14" effort="40.0" velocity="1.5"/>
 			<origin xyz="0 0 0.04" rpy="0 0 0"/>
+			<dynamics damping="1.0" friction="0.5"/>
 		</joint>
+		<link name="end_effector_tool_mount">
+			<visual>
+			<geometry><cylinder radius="0.05" length="0.02"/></geometry>
+			<material name="blue"/>
+			</visual>
+			<collision>
+			<geometry><cylinder radius="0.05" length="0.02"/></geometry>
+			</collision>
+			<!-- Tool mount plate (0.3 kg) -->
+			<xacro:cylinder_inertial mass="0.3" radius="0.05" length="0.02">
+			<origin xyz="0 0 0" rpy="0 0 0"/>
+			</xacro:cylinder_inertial>
+		</link>
 	</xacro:macro>
 </robot>

File: harvest_description/urdf/mech/rail.urdf.xacro (robot description, xacro)
@@ -2,31 +2,33 @@
 <robot xmlns:xacro="http://www.ros.org/wiki/xacro">
 	<xacro:macro name="rail" params="parent_link">
-		<link name="rail_link">
-			<visual>
-				<geometry>
-					<box size="2.0 0.1 0.05"/>
-				</geometry>
-				<material name="silver"/>
-			</visual>
-		</link>
+		<!-- WORLD ANCHOR AND RAIL -->
+		<!-- The rail macro owns the single world link used by the whole robot. -->
+		<link name="world"/>
 		<joint name="world_to_rail" type="fixed">
-			<parent link="${parent_link}"/>
+			<parent link="world"/>
 			<child link="rail_link"/>
 			<origin xyz="0 0 0" rpy="0 0 0"/>
 		</joint>
-		<link name="base_link">
+		<link name="rail_link">
 			<visual>
-				<geometry>
-					<cylinder radius="0.1" length="0.1"/>
-				</geometry>
-				<material name="blue"/>
+			<geometry><box size="2.0 0.1 0.05"/></geometry>
+			<material name="silver"/>
 			</visual>
+			<collision>
+			<geometry><box size="2.0 0.1 0.05"/></geometry>
+			</collision>
+			<!-- Heavy structural aluminum rail frame (15 kg) -->
+			<xacro:box_inertial mass="15.0" x="2.0" y="0.1" z="0.05">
+			<origin xyz="0 0 0" rpy="0 0 0"/>
+			</xacro:box_inertial>
 		</link>
+		<!-- 1. Rail Prismatic Joint -->
 		<joint name="rail_joint" type="prismatic">
 			<parent link="rail_link"/>
 			<child link="base_link"/>
 			<axis xyz="1 0 0"/>
-			<limit lower="-0.9" upper="0.9" effort="100.0" velocity="0.5"/>
+			<limit lower="-0.9" upper="0.9" effort="200.0" velocity="0.5"/>
 			<origin xyz="0 0 0.05" rpy="0 0 0"/>
+			<dynamics damping="10.0" friction="5.0"/>
 		</joint>
 	</xacro:macro>

File: harvest_description/urdf/mech/soft_gripper.urdf.xacro (robot description, xacro)
@@ -2,36 +2,52 @@
 <robot xmlns:xacro="http://www.ros.org/wiki/xacro">
 	<xacro:macro name="soft_gripper" params="parent_link">
-		<link name="camera_link">
-			<visual>
-				<geometry>
-					<box size="0.03 0.03 0.02"/>
-				</geometry>
-				<material name="red"/>
-			</visual>
-		</link>
+				<!-- CAMERA AND 3 FINGER GRIPPER -->
+		<!-- The tool mount is the attachment point for the camera and fingers. -->
+		<!-- Eye-in-Hand Camera Mount -->
 		<joint name="camera_joint" type="fixed">
-			<parent link="${parent_link}"/>
+			<parent link="end_effector_tool_mount"/>
 			<child link="camera_link"/>
 			<origin xyz="0.06 0 0.02" rpy="0 0 0"/>
 		</joint>
-		<xacro:macro name="finger" params="index angle">
-			<link name="finger_link_${index}">
-				<visual>
-					<origin xyz="0 0 0.04" rpy="0 0 0"/>
-					<geometry>
-						<box size="0.01 0.015 0.08"/>
-					</geometry>
-					<material name="green"/>
-				</visual>
+		<link name="camera_link">
+			<visual>
+			<geometry><box size="0.03 0.03 0.02"/></geometry>
+			<material name="red"/>
+			</visual>
+			<collision>
+			<geometry><box size="0.03 0.03 0.02"/></geometry>
+			</collision>
+			<!-- Lightweight camera module (0.05 kg / 50 grams) -->
+			<xacro:box_inertial mass="0.05" x="0.03" y="0.03" z="0.02">
+			<origin xyz="0 0 0" rpy="0 0 0"/>
+			</xacro:box_inertial>
+		</link>
+		<!-- Gripper Finger Macro -->
+		<xacro:macro name="finger" params="prefix yaw_angle">
+			<joint name="finger_joint_${prefix}" type="fixed">
+			<parent link="end_effector_tool_mount"/>
+			<child link="finger_link_${prefix}"/>
+			<origin xyz="${0.03 * cos(yaw_angle)} ${0.03 * sin(yaw_angle)} 0.02" rpy="0 0.2 ${yaw_angle}"/>
+			</joint>
+			<link name="finger_link_${prefix}">
+			<visual>
+				<origin xyz="0 0 0.04" rpy="0 0 0"/>
+				<geometry><box size="0.01 0.015 0.08"/></geometry>
+				<material name="green"/>
+			</visual>
+			<collision>
+				<origin xyz="0 0 0.04" rpy="0 0 0"/>
+				<geometry><box size="0.01 0.015 0.08"/></geometry>
+			</collision>
+			<!-- Ultra-lightweight soft silicone/rubber finger strand (0.02 kg / 20 grams) -->
+			<xacro:box_inertial mass="0.02" x="0.01" y="0.015" z="0.08">
+				<origin xyz="0 0 0.04" rpy="0 0 0"/>
+			</xacro:box_inertial>
 			</link>
-			<joint name="finger_joint_${index}" type="fixed">
-				<parent link="${parent_link}"/>
-				<child link="finger_link_${index}"/>
-				<origin xyz="${0.03 * cos(angle)} ${0.03 * sin(angle)} 0.02" rpy="0 0.2 ${angle}"/>
-			</joint>
 		</xacro:macro>
-		<xacro:finger index="1" angle="0.0"/>
-		<xacro:finger index="2" angle="2.094"/>
-		<xacro:finger index="3" angle="4.188"/>
+		<!-- Instantiate the 3 soft fingers -->
+		<xacro:finger prefix="1" yaw_angle="0.0"/>
+		<xacro:finger prefix="2" yaw_angle="2.094"/>
+		<xacro:finger prefix="3" yaw_angle="4.188"/>
 	</xacro:macro>
 </robot>

File: harvest_description/urdf/robots/harvest_280.urdf.xacro (robot description, xacro)
@@ -1,4 +1,27 @@
 <?xml version="1.0"?>
 <robot xmlns:xacro="http://www.ros.org/wiki/xacro" name="harvest_280">
+  <!-- Enable only when a working Gazebo ros2_control backend is available. -->
+  <xacro:arg name="use_gz_control" default="false"/>
+  <!-- INERTIAL MATH MACROS -->
+  <!-- Solid Cylinder Inertia Formula -->
+  <xacro:macro name="cylinder_inertial" params="mass radius length *origin">
+    <inertial>
+      <xacro:insert_block name="origin"/>
+      <mass value="${mass}"/>
+      <inertia ixx="${(1/12) * mass * (3*radius*radius + length*length)}" ixy="0.0" ixz="0.0"
+               iyy="${(1/12) * mass * (3*radius*radius + length*length)}" iyz="0.0"
+               izz="${(1/2) * mass * radius * radius}"/>
+    </inertial>
+  </xacro:macro>
+  <!-- Solid Box Inertia Formula -->
+  <xacro:macro name="box_inertial" params="mass x y z *origin">
+    <inertial>
+      <xacro:insert_block name="origin"/>
+      <mass value="${mass}"/>
+      <inertia ixx="${(1/12) * mass * (y*y + z*z)}" ixy="0.0" ixz="0.0"
+               iyy="${(1/12) * mass * (x*x + z*z)}" iyz="0.0"
+               izz="${(1/12) * mass * (x*x + y*y)}"/>
+    </inertial>
+  </xacro:macro>
   <xacro:include filename="$(find harvest_description)/urdf/mech/rail.urdf.xacro"/>
   <xacro:include filename="$(find harvest_description)/urdf/mech/harvest_arm.urdf.xacro"/>
@@ -9,7 +32,54 @@
   <material name="green"><color rgba="0.0 0.8 0.0 1.0"/></material>
   <material name="red"><color rgba="0.8 0.0 0.0 1.0"/></material>
-  <link name="world"/>
   <xacro:rail parent_link="world"/>
   <xacro:harvest_arm parent_link="base_link"/>
   <xacro:soft_gripper parent_link="end_effector_tool_mount"/>
+  <!-- GAZEBO SIMULATION SYSTEM PLUGIN -->
+  <!-- Keep the visual simulation independent from ros2_control startup. -->
+  <xacro:if value="$(arg use_gz_control)">
+    <gazebo>
+      <plugin filename="gz_ros2_control-system" name="gz_ros2_control::GazeboSimROS2ControlPlugin">
+        <parameters>$(find harvest_description)/urdf/control/robot_controllers.yaml</parameters>
+      </plugin>
+    </gazebo>
+  </xacro:if>
+  <!-- ROS2_CONTROL HARDWARE INTERFACE DEFINITION -->
+  <!-- These interfaces are included only for the opt-in controlled launch. -->
+  <xacro:if value="$(arg use_gz_control)">
+    <ros2_control name="GazeboSimSystem" type="system">
+    <hardware>
+      <plugin>gz_ros2_control/GazeboSimSystem</plugin>
+    </hardware>
+    <!-- 1. Rail Linear Actuator -->
+    <joint name="rail_joint">
+      <command_interface name="position"/>
+      <state_interface name="position"/>
+    </joint>
+    <!-- 2. Base Turn-table (Yaw) -->
+    <joint name="base_joint">
+      <command_interface name="position"/>
+      <state_interface name="position"/>
+    </joint>
+    <!-- 3. Shoulder (Pitch) -->
+    <joint name="shoulder_joint">
+      <command_interface name="position"/>
+      <state_interface name="position"/>
+    </joint>
+    <!-- 4. Elbow (Pitch) -->
+    <joint name="elbow_joint">
+      <command_interface name="position"/>
+      <state_interface name="position"/>
+    </joint>
+    <!-- 5. Wrist Pitch -->
+    <joint name="wrist_pitch_joint">
+      <command_interface name="position"/>
+      <state_interface name="position"/>
+    </joint>
+    <!-- 6. Wrist Roll -->
+    <joint name="wrist_roll_joint">
+      <command_interface name="position"/>
+      <state_interface name="position"/>
+    </joint>
+    </ros2_control>
+  </xacro:if>
 </robot>

Commit message: Added physics properties to the robot description. This includes collision and inertia properties for the robot links, which are essential for accurate physics simulation in Gazebo. The changes also include updates to the launch files and package dependencies to support these new features. Still struggling with moving the robot in Gazebo.

File: harvest_description/urdf/mech/harvest_arm.urdf.xacro (robot description, xacro)
@@ -1,5 +1,6 @@
 <?xml version="1.0"?>
 <robot xmlns:xacro="http://www.ros.org/wiki/xacro">
-	<xacro:macro name="harvest_arm" params="parent_link">
+	<xacro:include filename="$(find harvest_description)/urdf/robot_utils.urdf.xacro"/>
+	<xacro:macro name="harvest_arm">
 		  <!-- ARM STRUCTURE -->
 		<!-- The arm is attached to the rail carriage through base_link. -->
@@ -68,5 +69,5 @@
 		<joint name="elbow_joint" type="revolute">
 			<parent link="elbow_link"/>
-			<child xacro:name="wrist_pitch_link" link="wrist_pitch_link"/>
+			<child link="wrist_pitch_link"/>
 			<axis xyz="0 1 0"/>
 			<limit lower="-2.0" upper="2.0" effort="100.0" velocity="1.0"/>
@@ -74,5 +75,5 @@
 			<dynamics damping="3.0" friction="1.0"/>
 		</joint>
-		<!-- ================= Universal Wrist (Pitch-Roll) ================= -->
+		<!-- UNIVERSAL WRIST (PITCH-ROLL) -->
 		<link name="wrist_pitch_link">
 			<visual>

File: harvest_description/urdf/mech/rail.urdf.xacro (robot description, xacro)
@@ -1,5 +1,6 @@
 <?xml version="1.0"?>
 <robot xmlns:xacro="http://www.ros.org/wiki/xacro">
-	<xacro:macro name="rail" params="parent_link">
+	<xacro:include filename="$(find harvest_description)/urdf/robot_utils.urdf.xacro"/>
+	<xacro:macro name="rail">
 		<!-- WORLD ANCHOR AND RAIL -->
 		<!-- The rail macro owns the single world link used by the whole robot. -->

File: harvest_description/urdf/mech/soft_gripper.urdf.xacro (robot description, xacro)
@@ -1,6 +1,7 @@
 <?xml version="1.0"?>
 <robot xmlns:xacro="http://www.ros.org/wiki/xacro">
-	<xacro:macro name="soft_gripper" params="parent_link">
-				<!-- CAMERA AND 3 FINGER GRIPPER -->
+	<xacro:include filename="$(find harvest_description)/urdf/robot_utils.urdf.xacro"/>
+	<xacro:macro name="soft_gripper">
+		<!-- CAMERA AND 3 FINGER GRIPPER -->
 		<!-- The tool mount is the attachment point for the camera and fingers. -->
 		<!-- Eye-in-Hand Camera Mount -->
