Commit message: Fixing the simplified URDF from the original CAD model. Joints are still misplaced, but the model is now more accurate.

File: harvest_description/urdf/mech/harvest_arm.urdf.xacro (robot description, xacro)
@@ -1,136 +1,272 @@
 <?xml version="1.0"?>
 <robot xmlns:xacro="http://www.ros.org/wiki/xacro">
-	<xacro:include filename="$(find harvest_description)/urdf/robot_utils.urdf.xacro"/>
-	<xacro:macro name="harvest_arm">
-		  <!-- ARM STRUCTURE -->
-		<!-- The arm is attached to the rail carriage through base_link. -->
-		<link name="base_link">
-			<visual>
-			<geometry><cylinder radius="0.1" length="0.1"/></geometry>
-			<material name="blue"/>
-			</visual>
-			<collision>
-			<geometry><cylinder radius="0.1" length="0.1"/></geometry>
-			</collision>
-			<!-- Solid motor base carriage housing (5 kg) -->
-			<xacro:cylinder_inertial mass="5.0" radius="0.1" length="0.1">
-			<origin xyz="0 0 0" rpy="0 0 0"/>
-			</xacro:cylinder_inertial>
-		</link>
-		<!-- 2. Base Revolute Joint (Yaw) -->
-		<joint name="base_joint" type="revolute">
-			<parent link="base_link"/>
-			<child link="shoulder_link"/>
-			<axis xyz="0 0 1"/>
-			<limit lower="-3.14" upper="3.14" effort="150.0" velocity="1.0"/>
-			<origin xyz="0 0 0.05" rpy="0 0 0"/>
-			<dynamics damping="5.0" friction="2.0"/>
-		</joint>
-		<link name="shoulder_link">
-			<visual>
-			<origin xyz="0 0 0.2" rpy="0 0 0"/>
-			<geometry><cylinder radius="0.05" length="0.4"/></geometry>
-			<material name="silver"/>
-			</visual>
-			<collision>
-			<origin xyz="0 0 0.2" rpy="0 0 0"/>
-			<geometry><cylinder radius="0.05" length="0.4"/></geometry>
-			</collision>
-			<!-- Carbon fiber/aluminum lightweight link (2.5 kg) -->
-			<xacro:cylinder_inertial mass="2.5" radius="0.05" length="0.4">
-			<origin xyz="0 0 0.2" rpy="0 0 0"/>
-			</xacro:cylinder_inertial>
-		</link>
-		<!-- 3. Shoulder Revolute Joint (Pitch) -->
-		<joint name="shoulder_joint" type="revolute">
-			<parent link="shoulder_link"/>
-			<child link="elbow_link"/>
-			<axis xyz="0 1 0"/>
-			<limit lower="-1.57" upper="1.57" effort="150.0" velocity="1.0"/>
-			<origin xyz="0 0 0.4" rpy="0 0 0"/>
-			<dynamics damping="5.0" friction="2.0"/>
-		</joint>
-		<link name="elbow_link">
-			<visual>
-			<origin xyz="0 0 0.2" rpy="0 0 0"/>
-			<geometry><cylinder radius="0.04" length="0.4"/></geometry>
-			<material name="silver"/>
-			</visual>
-			<collision>
-			<origin xyz="0 0 0.2" rpy="0 0 0"/>
-			<geometry><cylinder radius="0.04" length="0.4"/></geometry>
-			</collision>
-			<!-- Upper arm link (2.0 kg) -->
-			<xacro:cylinder_inertial mass="2.0" radius="0.04" length="0.4">
-			<origin xyz="0 0 0.2" rpy="0 0 0"/>
-			</xacro:cylinder_inertial>
-		</link>
-		<!-- 4. Elbow Revolute Joint (Pitch) -->
-		<joint name="elbow_joint" type="revolute">
-			<parent link="elbow_link"/>
-			<child link="wrist_pitch_link"/>
-			<axis xyz="0 1 0"/>
-			<limit lower="-2.0" upper="2.0" effort="100.0" velocity="1.0"/>
-			<origin xyz="0 0 0.4" rpy="0 0 0"/>
-			<dynamics damping="3.0" friction="1.0"/>
-		</joint>
-		<!-- UNIVERSAL WRIST (PITCH-ROLL) -->
-		<link name="wrist_pitch_link">
-			<visual>
-			<geometry><cylinder radius="0.03" length="0.06"/></geometry>
-			<material name="blue"/>
-			</visual>
-			<collision>
-			<geometry><cylinder radius="0.03" length="0.06"/></geometry>
-			</collision>
-			<!-- Small pitch motor housing (0.8 kg) -->
-			<xacro:cylinder_inertial mass="0.8" radius="0.03" length="0.06">
-			<origin xyz="0 0 0" rpy="0 0 0"/>
-			</xacro:cylinder_inertial>
-		</link>
-		<!-- 5. Wrist Joint 1 (Pitch) -->
-		<joint name="wrist_pitch_joint" type="revolute">
-			<parent link="wrist_pitch_link"/>
-			<child link="wrist_roll_link"/>
-			<axis xyz="0 1 0"/>
-			<limit lower="-1.57" upper="1.57" effort="40.0" velocity="1.5"/>
-			<origin xyz="0 0 0.05" rpy="0 0 0"/>
-			<dynamics damping="1.0" friction="0.5"/>
-		</joint>
-		<link name="wrist_roll_link">
-			<visual>
-			<geometry><cylinder radius="0.03" length="0.04"/></geometry>
-			<material name="green"/>
-			</visual>
-			<collision>
-			<geometry><cylinder radius="0.03" length="0.04"/></geometry>
-			</collision>
-			<!-- Small roll motor housing (0.5 kg) -->
-			<xacro:cylinder_inertial mass="0.5" radius="0.03" length="0.04">
-			<origin xyz="0 0 0" rpy="0 0 0"/>
-			</xacro:cylinder_inertial>
-		</link>
-		<!-- 6. Wrist Joint 2 (Roll) -->
-		<joint name="wrist_roll_joint" type="revolute">
-			<parent link="wrist_roll_link"/>
-			<child link="end_effector_tool_mount"/>
-			<axis xyz="0 0 1"/>
-			<limit lower="-3.14" upper="3.14" effort="40.0" velocity="1.5"/>
-			<origin xyz="0 0 0.04" rpy="0 0 0"/>
-			<dynamics damping="1.0" friction="0.5"/>
-		</joint>
-		<link name="end_effector_tool_mount">
-			<visual>
-			<geometry><cylinder radius="0.05" length="0.02"/></geometry>
-			<material name="blue"/>
-			</visual>
-			<collision>
-			<geometry><cylinder radius="0.05" length="0.02"/></geometry>
-			</collision>
-			<!-- Tool mount plate (0.3 kg) -->
-			<xacro:cylinder_inertial mass="0.3" radius="0.05" length="0.02">
-			<origin xyz="0 0 0" rpy="0 0 0"/>
-			</xacro:cylinder_inertial>
-		</link>
-	</xacro:macro>
+  <xacro:include filename="$(find harvest_description)/urdf/robot_utils.urdf.xacro"/>
+  <!-- CAD actuator components are kept visual-only; existing collision bodies
+       stay lightweight and predictable for Gazebo contact and dynamics. -->
+  <!--
+    Each stage's housing transforms are expressed from its CAD output-drive
+    frame. The output pin itself belongs to the child link, so it moves with
+    the connected link instead of remaining fixed to the gearbox housing.
+  -->
+  <xacro:macro name="actuator_housing_visuals"
+               params="xyz housing_rpy internal_rpy">
+    <visual>
+      <origin xyz="${xyz}" rpy="${housing_rpy}"/>
+      <geometry><mesh filename="package://harvest_description/meshes/external_housing.gltf"/></geometry>
+    </visual>
+    <visual>
+      <origin xyz="${xyz}" rpy="${internal_rpy}"/>
+      <geometry><mesh filename="package://harvest_description/meshes/gearbox_housing.gltf"/></geometry>
+    </visual>
+    <visual>
+      <origin xyz="${xyz}" rpy="${internal_rpy}"/>
+      <geometry><mesh filename="package://harvest_description/meshes/nema17_smal.gltf"/></geometry>
+    </visual>
+  </xacro:macro>
+  <xacro:macro name="output_drive_visual" params="xyz rpy">
+    <visual>
+      <origin xyz="${xyz}" rpy="${rpy}"/>
+      <geometry><mesh filename="package://harvest_description/meshes/exterior_output_drive.gltf"/></geometry>
+    </visual>
+  </xacro:macro>
+  <xacro:macro name="harvest_arm">
+    <!--
+      The actuator sheet specifies a 200 g turret pedestal and five 575 g
+      actuators. The base link carries the pedestal and yaw actuator together.
+    -->
+    <link name="base_link">
+      <visual>
+        <!-- Raise the CAD's bottom-at-Z=0.108 mesh datum to the carriage top. -->
+        <origin xyz="-0.004 0.0134887 0.108" rpy="0 0 0"/>
+        <geometry><mesh filename="package://harvest_description/meshes/base_pcb_box.gltf"/></geometry>
+      </visual>
+      <!-- CAD yaw housing sits below the output frame; the pin rotates with shoulder_link. -->
+      <xacro:actuator_housing_visuals xyz="0 0 0.071"
+                                      housing_rpy="0 0 0"
+                                      internal_rpy="0 0 -2.83984"/>
+      <collision>
+        <origin xyz="0.03 0 0.054" rpy="0 0 0"/>
+        <geometry><box size="0.16 0.10 0.108"/></geometry>
+      </collision>
+      <inertial>
+        <origin xyz="0 0 0.05" rpy="0 0 0"/>
+        <mass value="0.775"/>
+        <inertia ixx="0.001230" ixy="0" ixz="0"
+                 iyy="0.001230" iyz="0" izz="0.001172"/>
+      </inertial>
+    </link>
+    <!-- The yaw axis sits at the top of the 108 mm pedestal, not in the rail. -->
+    <joint name="base_joint" type="revolute">
+      <parent link="base_link"/>
+      <child link="shoulder_link"/>
+      <origin xyz="0 0 0.108" rpy="0 0 0"/>
+      <axis xyz="0 0 1"/>
+      <limit lower="-3.14159" upper="3.14159" effort="3.92" velocity="1.0"/>
+      <dynamics damping="0.2" friction="0.05"/>
+    </joint>
+    <!-- J1 shoulder actuator (575 g), mounted at the first pitch axis. -->
+    <link name="shoulder_link">
+      <!-- The wide face of the yaw output pin faces outward from the turret. -->
+      <xacro:output_drive_visual xyz="0 0 -0.037" rpy="0 0 2.23158"/>
+      <visual>
+        <!-- The CAD pedestal rises from the base yaw output to the shoulder. -->
+        <origin xyz="-0.013783 -0.002826 0.002" rpy="0 0 1.48478"/>
+        <geometry><mesh filename="package://harvest_description/meshes/base_to_link.gltf"/></geometry>
+      </visual>
+      <!-- Housing parts are CAD-aligned to the shoulder output frame at z=0.096. -->
+      <xacro:actuator_housing_visuals xyz="0 0.037 0.096"
+                                      housing_rpy="1.5708 -1.5708 0"
+                                      internal_rpy="1.5708 1.26905 0"/>
+      <collision>
+        <origin xyz="0 0 0.096" rpy="0 0 0"/>
+        <geometry><cylinder radius="0.040" length="0.045"/></geometry>
+      </collision>
+      <inertial>
+        <origin xyz="0 0 0.096" rpy="1.5708 0 0"/>
+        <mass value="0.575"/>
+        <inertia ixx="0.000327" ixy="0" ixz="0"
+                 iyy="0.000327" iyz="0" izz="0.000460"/>
+      </inertial>
+    </link>
+    <!-- Link 1 is 150 mm center-to-center; its 100 g mass is from the sheet. -->
+    <joint name="shoulder_joint" type="revolute">
+      <parent link="shoulder_link"/>
+      <child link="elbow_link"/>
+      <!-- A zero shoulder angle now points the arm upward for a safe spawn pose. -->
+      <origin xyz="0 0 0.096" rpy="0 -1.5708 0"/>
+      <axis xyz="0 1 0"/>
+      <limit lower="-1.5708" upper="1.5708" effort="3.92" velocity="1.0"/>
+      <dynamics damping="0.2" friction="0.05"/>
+    </joint>
+    <link name="elbow_link">
+      <!-- This shoulder pin is on the moving link, with its broad face outward. -->
+      <xacro:output_drive_visual xyz="0 0.037 0"
+                                 rpy="1.5708 -0.40657 0"/>
+      <visual>
+        <!-- Rotate around the pin axis; origin compensation keeps the small hole fixed. -->
+        <origin xyz="-0.060000 -0.028000 -0.013489"
+                rpy="-1.570799 -0.000001 -1.570795"/>
+        <!-- Full CAD scale restores both end-hole diameters for the pin fits. -->
+        <geometry><mesh filename="package://harvest_description/meshes/joint_to_joint.gltf"
+                        scale="1 1 1"/></geometry>
+      </visual>
+      <collision>
+        <origin xyz="0.075 0 0" rpy="0 0 0"/>
+        <geometry><box size="0.15 0.035 0.025"/></geometry>
+      </collision>
+      <inertial>
+        <origin xyz="0.075 0 0" rpy="0 0 0"/>
+        <mass value="0.10"/>
+        <inertia ixx="0.00001917" ixy="0" ixz="0"
+                 iyy="0.00019010" iyz="0" izz="0.00019354"/>
+      </inertial>
+    </link>
+    <!-- J2 is at the end of link 1; its actuator mass is kept at the joint. -->
+    <joint name="elbow_actuator_mount" type="fixed">
+      <parent link="elbow_link"/>
+      <child link="elbow_actuator_link"/>
+      <origin xyz="0.15 0 0" rpy="0 0 0"/>
+    </joint>
+    <link name="elbow_actuator_link">
+      <!-- CAD elbow housing; its output pin is attached to wrist_pitch_link. -->
+      <xacro:actuator_housing_visuals xyz="0 0.037 0"
+                                      housing_rpy="1.5708 0 0"
+                                      internal_rpy="-1.5708 0.30175 -3.14159"/>
+      <collision>
+        <geometry><box size="0.065 0.060 0.045"/></geometry>
+      </collision>
+      <inertial>
+        <mass value="0.575"/>
+        <inertia ixx="0.0003586" ixy="0" ixz="0"
+                 iyy="0.0003981" iyz="0" izz="0.0003813"/>
+      </inertial>
+    </link>
+    <!-- Link 2 is the second 150 mm link, with its 100 g structural mass. -->
+    <joint name="elbow_joint" type="revolute">
+      <parent link="elbow_actuator_link"/>
+      <child link="wrist_pitch_link"/>
+      <axis xyz="0 1 0"/>
+      <limit lower="-2.0" upper="2.0" effort="2.94" velocity="1.0"/>
+      <dynamics damping="0.2" friction="0.05"/>
+    </joint>
+    <link name="wrist_pitch_link">
+      <xacro:output_drive_visual xyz="0 0.037 0"
+                                 rpy="1.5708 -1.02212 0"/>
+      <visual>
+        <!-- Rotate around the pin axis; origin compensation keeps the small hole fixed. -->
+        <origin xyz="-0.060000 -0.028000 -0.013489"
+                rpy="-1.570802 0.000000 -1.570796"/>
+        <!-- Match the first connector's CAD-scale end holes and pin fit. -->
+        <geometry><mesh filename="package://harvest_description/meshes/joint_to_joint.gltf"
+                        scale="1 1 1"/></geometry>
+      </visual>
+      <collision>
+        <origin xyz="0.075 0 0" rpy="0 0 0"/>
+        <geometry><box size="0.15 0.032 0.024"/></geometry>
+      </collision>
+      <inertial>
+        <origin xyz="0.075 0 0" rpy="0 0 0"/>
+        <mass value="0.10"/>
+        <inertia ixx="0.00001333" ixy="0" ixz="0"
+                 iyy="0.00019230" iyz="0" izz="0.00019520"/>
+      </inertial>
+    </link>
+    <!-- J3 is the upper elbow actuator at the end of link 2. -->
+    <joint name="wrist_pitch_actuator_mount" type="fixed">
+      <parent link="wrist_pitch_link"/>
+      <child link="wrist_pitch_actuator_link"/>
+      <origin xyz="0.15 0 0" rpy="0 0 0"/>
+    </joint>
+    <link name="wrist_pitch_actuator_link">
+      <!-- CAD wrist-pitch housing; the output pin moves with wrist_roll_link. -->
+      <xacro:actuator_housing_visuals xyz="0 0.037 0"
+                                      housing_rpy="1.5708 0 0"
+                                      internal_rpy="-1.5708 0.30175 -3.14159"/>
+      <collision>
+        <geometry><box size="0.065 0.060 0.045"/></geometry>
+      </collision>
+      <inertial>
+        <mass value="0.575"/>
+        <inertia ixx="0.0003586" ixy="0" ixz="0"
+                 iyy="0.0003981" iyz="0" izz="0.0003813"/>
+      </inertial>
+    </link>
+    <!-- Link 3 is the 150 g, 150 mm wrist link from the actuator sheet. -->
+    <joint name="wrist_pitch_joint" type="revolute">
+      <parent link="wrist_pitch_actuator_link"/>
+      <child link="wrist_roll_link"/>
+      <axis xyz="0 1 0"/>
+      <limit lower="-1.5708" upper="1.5708" effort="0.956" velocity="1.5"/>
+      <dynamics damping="0.1" friction="0.02"/>
+    </joint>
+    <link name="wrist_roll_link">
+      <xacro:output_drive_visual xyz="0 0.037 0"
+                                 rpy="1.5708 0.607152 0"/>
+      <visual>
+        <!--
+          The CAD link runs along its mesh Y axis. Keep that axis exactly on the
+          arm's X axis and shift its end ring onto the fourth gearbox pin face.
+          The pitch is a clocking rotation about the link axis for hole alignment.
+        -->
+        <origin xyz="0.011667 -0.026998 -0.363404"
+                rpy="0 0 -1.5708"/>
+        <geometry><mesh filename="package://harvest_description/meshes/Part_4.gltf"/></geometry>
+      </visual>
+      <collision>
+        <origin xyz="0.075 0 0" rpy="0 0 0"/>
+        <geometry><box size="0.15 0.045 0.025"/></geometry>
+      </collision>
+      <inertial>
+        <origin xyz="0.075 0 0" rpy="0 0 0"/>
+        <mass value="0.15"/>
+        <inertia ixx="0.00003313" ixy="0" ixz="0"
+                 iyy="0.00028906" iyz="0" izz="0.00030656"/>
+      </inertial>
+    </link>
+    <!-- J4 rolls the tool about the arm's longitudinal axis. -->
+    <joint name="wrist_roll_actuator_mount" type="fixed">
+      <parent link="wrist_roll_link"/>
+      <child link="wrist_roll_actuator_link"/>
+      <origin xyz="0.15 0 0" rpy="0 0 0"/>
+    </joint>
+    <link name="wrist_roll_actuator_link">
+      <!-- End housing faces down; the CAD-aligned output pin is on the tool mount. -->
+      <xacro:actuator_housing_visuals xyz="-0.037 0 0"
+                                      housing_rpy="0 1.5708 0"
+                                      internal_rpy="-1.5708 -1.26905 -1.5708"/>
+      <collision>
+        <geometry><box size="0.065 0.060 0.045"/></geometry>
+      </collision>
+      <inertial>
+        <mass value="0.575"/>
+        <inertia ixx="0.0003586" ixy="0" ixz="0"
+                 iyy="0.0003981" iyz="0" izz="0.0003813"/>
+      </inertial>
+    </link>
+    <joint name="wrist_roll_joint" type="revolute">
+      <parent link="wrist_roll_actuator_link"/>
+      <child link="end_effector_tool_mount"/>
+      <!-- Place the tool flange on the output face, above the housing when upright. -->
+      <origin xyz="0.02 0 0" rpy="0 0 0"/>
+      <axis xyz="1 0 0"/>
+      <limit lower="-3.14159" upper="3.14159" effort="2.94" velocity="1.5"/>
+      <dynamics damping="0.1" friction="0.02"/>
+    </joint>
+    <link name="end_effector_tool_mount">
+      <xacro:output_drive_visual xyz="-0.057 0 0"
+                                 rpy="1.5708 0.163976 1.5708"/>
+      <visual>
+        <geometry><cylinder radius="0.035" length="0.012"/></geometry>
+        <material name="silver"/>
+      </visual>
+      <collision>
+        <geometry><cylinder radius="0.035" length="0.012"/></geometry>
+      </collision>
+      <inertial>
+        <mass value="0.01"/>
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
File: harvest_description/urdf/mech/rail.urdf.xacro (robot description, xacro)
@@ -25,4 +25,6 @@
 		</link>
 		<!-- 1. Rail Prismatic Joint -->
+		<!-- The carriage frame is on the rail's upper face (half of its 50 mm
+		     thickness), so the carriage housing rests directly on the rail. -->
 		<joint name="rail_joint" type="prismatic">
 			<parent link="rail_link"/>
@@ -30,5 +32,5 @@
 			<axis xyz="1 0 0"/>
 			<limit lower="-0.9" upper="0.9" effort="200.0" velocity="0.5"/>
-			<origin xyz="0 0 0.05" rpy="0 0 0"/>
+			<origin xyz="0 0 0.025" rpy="0 0 0"/>
 			<dynamics damping="10.0" friction="5.0"/>
 		</joint>

File: harvest_description/urdf/mech/soft_gripper.urdf.xacro (robot description, xacro)
@@ -1,54 +1,53 @@
 <?xml version="1.0"?>
 <robot xmlns:xacro="http://www.ros.org/wiki/xacro">
-	<xacro:include filename="$(find harvest_description)/urdf/robot_utils.urdf.xacro"/>
-	<xacro:macro name="soft_gripper">
-		<!-- CAMERA AND 3 FINGER GRIPPER -->
-		<!-- The tool mount is the attachment point for the camera and fingers. -->
-		<!-- Eye-in-Hand Camera Mount -->
-		<joint name="camera_joint" type="fixed">
-			<parent link="end_effector_tool_mount"/>
-			<child link="camera_link"/>
-			<origin xyz="0.06 0 0.02" rpy="0 0 0"/>
-		</joint>
-		<link name="camera_link">
-			<visual>
-			<geometry><box size="0.03 0.03 0.02"/></geometry>
-			<material name="red"/>
-			</visual>
-			<collision>
-			<geometry><box size="0.03 0.03 0.02"/></geometry>
-			</collision>
-			<!-- Lightweight camera module (0.05 kg / 50 grams) -->
-			<xacro:box_inertial mass="0.05" x="0.03" y="0.03" z="0.02">
-			<origin xyz="0 0 0" rpy="0 0 0"/>
-			</xacro:box_inertial>
-		</link>
-		<!-- Gripper Finger Macro -->
-		<xacro:macro name="finger" params="prefix yaw_angle">
-			<joint name="finger_joint_${prefix}" type="fixed">
-			<parent link="end_effector_tool_mount"/>
-			<child link="finger_link_${prefix}"/>
-			<origin xyz="${0.03 * cos(yaw_angle)} ${0.03 * sin(yaw_angle)} 0.02" rpy="0 0.2 ${yaw_angle}"/>
-			</joint>
-			<link name="finger_link_${prefix}">
-			<visual>
-				<origin xyz="0 0 0.04" rpy="0 0 0"/>
-				<geometry><box size="0.01 0.015 0.08"/></geometry>
-				<material name="green"/>
-			</visual>
-			<collision>
-				<origin xyz="0 0 0.04" rpy="0 0 0"/>
-				<geometry><box size="0.01 0.015 0.08"/></geometry>
-			</collision>
-			<!-- Ultra-lightweight soft silicone/rubber finger strand (0.02 kg / 20 grams) -->
-			<xacro:box_inertial mass="0.02" x="0.01" y="0.015" z="0.08">
-				<origin xyz="0 0 0.04" rpy="0 0 0"/>
-			</xacro:box_inertial>
-			</link>
-		</xacro:macro>
-		<!-- Instantiate the 3 soft fingers -->
-		<xacro:finger prefix="1" yaw_angle="0.0"/>
-		<xacro:finger prefix="2" yaw_angle="2.094"/>
-		<xacro:finger prefix="3" yaw_angle="4.188"/>
-	</xacro:macro>
+  <xacro:include filename="$(find harvest_description)/urdf/robot_utils.urdf.xacro"/>
+  <xacro:macro name="soft_gripper">
+    <!-- This frame is mounted on the fourth gearbox output, above the blue link. -->
+    <!-- The camera sits on the rear of the mount, away from the grasping area. -->
+    <joint name="camera_joint" type="fixed">
+      <parent link="end_effector_tool_mount"/>
+      <child link="camera_link"/>
+      <origin xyz="0.0125 0.02 0.02" rpy="0 0 0"/>
+    </joint>
+    <link name="camera_link">
+      <visual>
+        <geometry><box size="0.035 0.035 0.025"/></geometry>
+        <material name="red"/>
+      </visual>
+      <collision>
+        <geometry><box size="0.035 0.035 0.025"/></geometry>
+      </collision>
+      <xacro:box_inertial mass="0.05" x="0.035" y="0.035" z="0.025">
+        <origin xyz="0 0 0" rpy="0 0 0"/>
+      </xacro:box_inertial>
+    </link>
+      <!-- Finger Template Macro (Instantiates 3 flexible grasping links at 120-degree patterns) -->
+    <!-- Each lightweight 80 mm finger extends forward along the arm's +X axis. -->
+    <xacro:macro name="finger" params="prefix angle">
+      <joint name="finger_joint_${prefix}" type="fixed">
+        <parent link="end_effector_tool_mount"/>
+        <child link="finger_link_${prefix}"/>
+        <origin xyz="0.005 ${0.025 * cos(angle)} ${0.025 * sin(angle)}"
+                rpy="${angle} 0 0"/>
+      </joint>
+      <link name="finger_link_${prefix}">
+        <visual>
+          <origin xyz="0.04 0 0" rpy="0 0 0"/>
+          <geometry><box size="0.08 0.012 0.012"/></geometry>
+          <material name="green"/>
+        </visual>
+        <collision>
+          <origin xyz="0.04 0 0" rpy="0 0 0"/>
+          <geometry><box size="0.08 0.012 0.012"/></geometry>
+        </collision>
+        <xacro:box_inertial mass="0.02" x="0.08" y="0.012" z="0.012">
+          <origin xyz="0.04 0 0" rpy="0 0 0"/>
+        </xacro:box_inertial>
+      </link>
+    </xacro:macro>
+    <!-- The fingers are spaced at 120-degree intervals -->
+    <xacro:finger prefix="1" angle="0.0"/>
+    <xacro:finger prefix="2" angle="2.094395"/>
+    <xacro:finger prefix="3" angle="4.188790"/>
+  </xacro:macro>
 </robot>

File: harvest_description/urdf/robots/harvest_full.urdf.xacro (robot description, xacro)
@@ -1,4 +1,4 @@
 <?xml version="1.0"?>
-<robot xmlns:xacro="http://www.ros.org/wiki/xacro" name="harvest_280">
+<robot xmlns:xacro="http://www.ros.org/wiki/xacro" name="harvest_robot">
   <xacro:include filename="$(find harvest_description)/urdf/mech/rail.urdf.xacro"/>
   <xacro:include filename="$(find harvest_description)/urdf/mech/harvest_arm.urdf.xacro"/>
