Commit message: Added twist action to the kinematics. Fixed the URDF so that the robot structure matches the 3D CAD model.

File: harvest_description/urdf/mech/harvest_arm.urdf.xacro (robot description, xacro)
@@ -75,5 +75,5 @@
       </visual>
       <!-- Housing parts are CAD-aligned to the shoulder output frame at z=0.096. -->
-      <xacro:actuator_housing_visuals xyz="0 0.037 0.096"
+      <xacro:actuator_housing_visuals xyz="0 0.045 0.061"
                                       housing_rpy="1.5708 -1.5708 0"
                                       internal_rpy="1.5708 1.26905 0"/>
@@ -94,5 +94,5 @@
       <child link="elbow_link"/>
       <!-- A zero shoulder angle now points the arm upward for a safe spawn pose. -->
-      <origin xyz="0 0 0.096" rpy="0 -1.5708 0"/>
+      <origin xyz="0 0 0.061" rpy="0 -1.5708 0"/>
       <axis xyz="0 1 0"/>
       <limit lower="-1.5708" upper="1.5708" effort="3.92" velocity="1.0"/>
@@ -228,5 +228,5 @@
       <parent link="wrist_roll_link"/>
       <child link="wrist_roll_actuator_link"/>
-      <origin xyz="0.15 0 0" rpy="0 0 0"/>
+      <origin xyz="0.14 -0.072 0" rpy="0 0 0"/>
     </joint>
     <link name="wrist_roll_actuator_link">
@@ -257,8 +257,10 @@
                                  rpy="1.5708 0.163976 1.5708"/>
       <visual>
+        <origin xyz="0 0 0" rpy="0 1.5708 0"/>
         <geometry><cylinder radius="0.035" length="0.012"/></geometry>
         <material name="silver"/>
       </visual>
       <collision>
+        <origin xyz="0 0 0" rpy="0 1.5708 0"/>
         <geometry><cylinder radius="0.035" length="0.012"/></geometry>
       </collision>

Commit message: Managed to fix the kinematics nodes. Updated the effort for all joint limit tags in the URDF. They were too low and the arm would sag, thus not reaching the target.

File: harvest_description/urdf/mech/harvest_arm.urdf.xacro (robot description, xacro)
@@ -57,4 +57,5 @@
     </link>
     <!-- The yaw axis sits at the top of the 108 mm pedestal, not in the rail. -->
+    <!-- J1 Base Yaw -->
     <joint name="base_joint" type="revolute">
       <parent link="base_link"/>
@@ -62,5 +63,6 @@
       <origin xyz="0 0 0.108" rpy="0 0 0"/>
       <axis xyz="0 0 1"/>
-      <limit lower="-3.14159" upper="3.14159" effort="3.92" velocity="1.0"/>
+      <!-- updated all joint limit tags so that arm does not sag under gravity. -->
+      <limit lower="-3.14159" upper="3.14159" effort="10.0" velocity="1.0"/>
       <dynamics damping="0.2" friction="0.05"/>
     </joint>
@@ -90,4 +92,5 @@
     </link>
     <!-- Link 1 is 150 mm center-to-center; its 100 g mass is from the sheet. -->
+    <!-- J2 Shoulder Pitch (Lifts the entire 2kg arm assembly) -->
     <joint name="shoulder_joint" type="revolute">
       <parent link="shoulder_link"/>
@@ -96,5 +99,5 @@
       <origin xyz="0 0 0.061" rpy="0 -1.5708 0"/>
       <axis xyz="0 1 0"/>
-      <limit lower="-1.5708" upper="1.5708" effort="3.92" velocity="1.0"/>
+      <limit lower="-1.5708" upper="1.5708" effort="15.0" velocity="1.0"/>
       <dynamics damping="0.2" friction="0.05"/>
     </joint>
@@ -143,9 +146,10 @@
     </link>
     <!-- Link 2 is the second 150 mm link, with its 100 g structural mass. -->
+    <!-- J3 Elbow Pitch (Lifts the forearm, two actuators, and gripper) -->
     <joint name="elbow_joint" type="revolute">
       <parent link="elbow_actuator_link"/>
       <child link="wrist_pitch_link"/>
       <axis xyz="0 1 0"/>
-      <limit lower="-2.0" upper="2.0" effort="2.94" velocity="1.0"/>
+      <limit lower="-2.0" upper="2.0" effort="10.0" velocity="1.0"/>
       <dynamics damping="0.2" friction="0.05"/>
     </joint>
@@ -193,9 +197,10 @@
     </link>
     <!-- Link 3 is the 150 g, 150 mm wrist link from the actuator sheet. -->
+    <!-- J4 Wrist Pitch (Lifts the roll actuator and gripper) -->
     <joint name="wrist_pitch_joint" type="revolute">
       <parent link="wrist_pitch_actuator_link"/>
       <child link="wrist_roll_link"/>
       <axis xyz="0 1 0"/>
-      <limit lower="-1.5708" upper="1.5708" effort="0.956" velocity="1.5"/>
+      <limit lower="-1.5708" upper="1.5708" effort="5.0" velocity="1.5"/>
       <dynamics damping="0.1" friction="0.02"/>
     </joint>
@@ -244,4 +249,5 @@
       </inertial>
     </link>
+    <!-- J5 Wrist Roll -->
     <joint name="wrist_roll_joint" type="revolute">
       <parent link="wrist_roll_actuator_link"/>
@@ -250,5 +256,5 @@
       <origin xyz="0.02 0 0" rpy="0 0 0"/>
       <axis xyz="1 0 0"/>
-      <limit lower="-3.14159" upper="3.14159" effort="2.94" velocity="1.5"/>
+      <limit lower="-3.14159" upper="3.14159" effort="5.0" velocity="1.5"/>
       <dynamics damping="0.1" friction="0.02"/>
     </joint>

Commit message: Added s-curve trajectory planning which has 7 time phases to calculate position, velocity, acceleration and jerk. Included scripts to generate graphs from the data parsed from the database of the simulation. Tuning PID and effort to reduce oscillations

File: harvest_description/urdf/mech/harvest_arm.urdf.xacro (robot description, xacro)
@@ -151,5 +151,5 @@
       <child link="wrist_pitch_link"/>
       <axis xyz="0 1 0"/>
-      <limit lower="-2.0" upper="2.0" effort="10.0" velocity="1.0"/>
+      <limit lower="-2.0" upper="2.0" effort="15.0" velocity="1.0"/>
       <dynamics damping="0.2" friction="0.05"/>
     </joint>

File: harvest_description/urdf/robots/harvest_full.urdf.xacro (robot description, xacro)
@@ -30,24 +30,30 @@
   <joint name="rail_joint">
       <command_interface name="position"><param name="min">-0.9</param><param name="max">0.9</param></command_interface>
+      <command_interface name="effort"/>
       <state_interface name="position"/><state_interface name="velocity"/><state_interface name="effort"/>
   </joint>
   <joint name="base_joint">
     <command_interface name="position"><param name="min">-3.14</param><param name="max">3.14</param></command_interface>
+    <command_interface name="effort"/>
     <state_interface name="position"/><state_interface name="velocity"/><state_interface name="effort"/>
   </joint>
   <joint name="shoulder_joint">
     <command_interface name="position"><param name="min">-1.57</param><param name="max">1.57</param></command_interface>
+    <command_interface name="effort"/>
     <state_interface name="position"/><state_interface name="velocity"/><state_interface name="effort"/>
   </joint>
   <joint name="elbow_joint">
     <command_interface name="position"><param name="min">-2.0</param><param name="max">2.0</param></command_interface>
+    <command_interface name="effort"/>
     <state_interface name="position"/><state_interface name="velocity"/><state_interface name="effort"/>
   </joint>
   <joint name="wrist_pitch_joint">
     <command_interface name="position"><param name="min">-1.57</param><param name="max">1.57</param></command_interface>
+    <command_interface name="effort"/>
     <state_interface name="position"/><state_interface name="velocity"/><state_interface name="effort"/>
   </joint>
   <joint name="wrist_roll_joint">
     <command_interface name="position"><param name="min">-3.14</param><param name="max">3.14</param></command_interface>
+    <command_interface name="effort"/>
     <state_interface name="position"/><state_interface name="velocity"/><state_interface name="effort"/>
   </joint>

Commit message: Additional comments to code Updated control loop frequency

File: harvest_description/urdf/mech/harvest_arm.urdf.xacro (robot description, xacro)
@@ -64,5 +64,5 @@
       <axis xyz="0 0 1"/>
       <!-- updated all joint limit tags so that arm does not sag under gravity. -->
-      <limit lower="-3.14159" upper="3.14159" effort="10.0" velocity="1.0"/>
+      <limit lower="-3.14159" upper="3.14159" effort="3.0" velocity="1.0"/>
       <dynamics damping="0.2" friction="0.05"/>
     </joint>
@@ -99,5 +99,5 @@
       <origin xyz="0 0 0.061" rpy="0 -1.5708 0"/>
       <axis xyz="0 1 0"/>
-      <limit lower="-1.5708" upper="1.5708" effort="15.0" velocity="1.0"/>
+      <limit lower="-1.5708" upper="1.5708" effort="3.0" velocity="1.0"/>
       <dynamics damping="0.2" friction="0.05"/>
     </joint>
@@ -151,5 +151,5 @@
       <child link="wrist_pitch_link"/>
       <axis xyz="0 1 0"/>
-      <limit lower="-2.0" upper="2.0" effort="15.0" velocity="1.0"/>
+      <limit lower="-2.0" upper="2.0" effort="3.0" velocity="1.0"/>
       <dynamics damping="0.2" friction="0.05"/>
     </joint>
@@ -202,5 +202,5 @@
       <child link="wrist_roll_link"/>
       <axis xyz="0 1 0"/>
-      <limit lower="-1.5708" upper="1.5708" effort="5.0" velocity="1.5"/>
+      <limit lower="-1.5708" upper="1.5708" effort="3.0" velocity="1.5"/>
       <dynamics damping="0.1" friction="0.02"/>
     </joint>
@@ -256,5 +256,5 @@
       <origin xyz="0.02 0 0" rpy="0 0 0"/>
       <axis xyz="1 0 0"/>
-      <limit lower="-3.14159" upper="3.14159" effort="5.0" velocity="1.5"/>
+      <limit lower="-3.14159" upper="3.14159" effort="3.0" velocity="1.5"/>
       <dynamics damping="0.1" friction="0.02"/>
     </joint>

Commit message: Tuned PIDs to the possible gain values. Kept effort true to physical robot by changing it to 4.0 for joints. Altered trajectory planner to reduce jerk which was causing aggressive shaking. Increased the controller loop rate to 2000 Hz to reduce violent robot shaking.

File: harvest_description/urdf/mech/harvest_arm.urdf.xacro (robot description, xacro)
@@ -64,5 +64,5 @@
       <axis xyz="0 0 1"/>
       <!-- updated all joint limit tags so that arm does not sag under gravity. -->
-      <limit lower="-3.14159" upper="3.14159" effort="3.0" velocity="1.0"/>
+      <limit lower="-3.14159" upper="3.14159" effort="4.0" velocity="1.0"/>
       <dynamics damping="0.2" friction="0.05"/>
     </joint>
@@ -99,5 +99,5 @@
       <origin xyz="0 0 0.061" rpy="0 -1.5708 0"/>
       <axis xyz="0 1 0"/>
-      <limit lower="-1.5708" upper="1.5708" effort="3.0" velocity="1.0"/>
+      <limit lower="-1.5708" upper="1.5708" effort="5.0" velocity="1.0"/>
       <dynamics damping="0.2" friction="0.05"/>
     </joint>
@@ -151,5 +151,5 @@
       <child link="wrist_pitch_link"/>
       <axis xyz="0 1 0"/>
-      <limit lower="-2.0" upper="2.0" effort="3.0" velocity="1.0"/>
+      <limit lower="-2.0" upper="2.0" effort="4.0" velocity="1.0"/>
       <dynamics damping="0.2" friction="0.05"/>
     </joint>
@@ -202,5 +202,5 @@
       <child link="wrist_roll_link"/>
       <axis xyz="0 1 0"/>
-      <limit lower="-1.5708" upper="1.5708" effort="3.0" velocity="1.5"/>
+      <limit lower="-1.5708" upper="1.5708" effort="4.0" velocity="1.5"/>
       <dynamics damping="0.1" friction="0.02"/>
     </joint>
@@ -256,5 +256,5 @@
       <origin xyz="0.02 0 0" rpy="0 0 0"/>
       <axis xyz="1 0 0"/>
-      <limit lower="-3.14159" upper="3.14159" effort="3.0" velocity="1.5"/>
+      <limit lower="-3.14159" upper="3.14159" effort="4.0" velocity="1.5"/>
       <dynamics damping="0.1" friction="0.02"/>
     </joint>

Commit message: Added gravity compensation to prevent joint from sagging or completely missing their targets. Updated effort values as well as PID gains to ensure that they match real world contraints and torques. Updated the trajectory planning script to try and improve time scaling. Joint values are still misaligned, thus the issue is unresolved.

File: harvest_description/urdf/mech/harvest_arm.urdf.xacro (robot description, xacro)
@@ -99,5 +99,5 @@
       <origin xyz="0 0 0.061" rpy="0 -1.5708 0"/>
       <axis xyz="0 1 0"/>
-      <limit lower="-1.5708" upper="1.5708" effort="5.0" velocity="1.0"/>
+      <limit lower="-1.5708" upper="1.5708" effort="5.60" velocity="1.0"/>
       <dynamics damping="0.2" friction="0.05"/>
     </joint>

Commit message: Changed some of the logic in the harvest ros2 nodes Filled in the README files Tuned PID gains again System is still oscillating

File: harvest_description/urdf/mech/harvest_arm.urdf.xacro (robot description, xacro)
@@ -99,5 +99,5 @@
       <origin xyz="0 0 0.061" rpy="0 -1.5708 0"/>
       <axis xyz="0 1 0"/>
-      <limit lower="-1.5708" upper="1.5708" effort="5.60" velocity="1.0"/>
+      <limit lower="-1.5708" upper="1.5708" effort="30.0" velocity="1.0"/>
       <dynamics damping="0.2" friction="0.05"/>
     </joint>
@@ -151,5 +151,5 @@
       <child link="wrist_pitch_link"/>
       <axis xyz="0 1 0"/>
-      <limit lower="-2.0" upper="2.0" effort="4.0" velocity="1.0"/>
+      <limit lower="-2.0" upper="2.0" effort="15.0" velocity="1.0"/>
       <dynamics damping="0.2" friction="0.05"/>
     </joint>
@@ -202,5 +202,5 @@
       <child link="wrist_roll_link"/>
       <axis xyz="0 1 0"/>
-      <limit lower="-1.5708" upper="1.5708" effort="4.0" velocity="1.5"/>
+      <limit lower="-1.5708" upper="1.5708" effort="10.0" velocity="1.5"/>
       <dynamics damping="0.1" friction="0.02"/>
     </joint>
